File: Switching_power_supply.kicad_sch (KiCad schematic)
At the start: 28 parts, among them J6 Conn_01x03_Pin, SW1 SW_DIP_x04, U3 AMS1117, U5 LM2596HVS-ADJRG

Commit message: moved sth and added hierarhical pins
Parts:
- removed C3, C4: 10uF, PCM_JLCPCB:C_0603, symbol PCM_JLCPCB-Capacitors:0603,10uF
- removed D2, D4, D5: SS510C, SS510C:SMC_L7.1-W6.2-LS8.1-RD, symbol SS510C:SS510C
- removed J6: Conn_01x03_Pin, Connector_PinHeader_2.54mm:PinHeader_1x03_P2.54mm_Vertical, symbol Connector:Conn_01x03_Pin
- removed U3: AMS1117, PCM_JLCPCB:SOT-223-3_L6.5-W3.4-P2.30-LS7.0-BR, symbol PCM_JLCPCB-Power:LDO, 3.3V, 1A
Connections:
- net U_reg renamed VOUT
- net sw-vin renamed VIN
Other:
- note removed: "3V3 LDO"
- note removed: "Connect 2-1 To use regulator 2-3 To bypas regulator and use Vin directly"
- note removed: "Diodes to drop voltage from chainbus max 48V to 46V for TMC5130A-TA to handle"
- note removed: "LM2596 Step-Down Regulator"
